File: pcb/rpi_ad7705.sch (EAGLE design)
At the start: 17 parts

Commit message: Updated circuit with an oscillator and new pin header.
Parts:
- removed SV1: RASPBERRY PI, con-lsta:FE13-2
- added C4: 0.1uF, capacitor-wima:C5/2.5
- added Q1: 2.4576 MHz, crystal:ASFL
- added SV5: (no value), con-lsta:FE20-2
Connections:
- removed net N$18: R9.1, SV4.3
- new net N$22: C1.+, U$1.REFIN+, U$2.VOUT
- net +3V3: now also C4.2, Q1.OE, Q1.VCC, SV2.4, SV3.4, SV5.1; no longer SV1.1, SV6.1
- net GND: now also C4.1, Q1.GND, SV5.39, SV5.6, SV6.1; no longer SV1.6
- net N$1: now also SV5.19; no longer SV1.19
- net N$15: now also R10.1, SV4.3; no longer R9.2, SV1.11
- net N$16: now also R9.2, SV5.31; no longer R10.1, SV1.12
- net N$17: now also R10.2, SV5.29; no longer R11.2, SV1.13
- net N$2: now also SV5.23; no longer SV1.23
- net N$20: now also R9.1; no longer R10.2
- net N$21: now also SV5.15; no longer SV1.15
- net N$3: now also Q1.FO; no longer SV1.7
- net N$4: now also SV5.24; no longer SV1.24
- net N$5: now also R11.2, SV5.37; no longer C1.+, SV2.4, SV3.4, U$1.REFIN+, U$2.VOUT
- net N$6: now also SV5.21; no longer SV1.21
Other:
- note added: "(C) 2014-2020 Bernd Porr"
- note removed: "(C) 2014 Bernd Porr"
- moved on the sheet: R10

Commit message: Switched the molex to the other side
Parts:
- removed SV6: 3.3V, jumper:JP1E
Connections:
- net +3V3: no longer SV6.2
- net GND: no longer SV6.1
Changed lines of the file:
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@@
 <part name="GND8" library="supply1" deviceset="GND" device=""/>
 <part name="C3" library="rcl" deviceset="CPOL-EU" device="TT2D7" value="1uF/tantalum"/>
-<part name="SV6" library="jumper" deviceset="JP1E" device="" value="3.3V"/>
-<part name="+3V5" library="supply1" deviceset="+3V3" device=""/>
 <part name="C1" library="rcl" deviceset="CPOL-EU" device="TT2D7" value="1uF/tantalum"/>
 <part name="SV2" library="con-lstb" deviceset="MA04-1" device=""/>
@@
 <part name="SV5" library="con-lsta" deviceset="FE20-2" device=""/>
 <part name="+3V7" library="supply1" deviceset="+3V3" device=""/>
-<part name="GND10" library="supply1" deviceset="GND" device=""/>
 <part name="GND11" library="supply1" deviceset="GND" device=""/>
 </parts>
@@
 <instance part="GND8" gate="1" x="91.44" y="20.32"/>
 <instance part="C3" gate="G$1" x="68.58" y="86.36"/>
-<instance part="SV6" gate="A" x="-33.02" y="68.58" rot="R90"/>
-<instance part="+3V5" gate="G$1" x="-22.86" y="78.74"/>
 <instance part="C1" gate="G$1" x="66.04" y="30.48"/>
 <instance part="SV2" gate="1" x="-35.56" y="38.1"/>
@@
 <instance part="SV5" gate="G$1" x="129.54" y="73.66" rot="MR90"/>
 <instance part="+3V7" gate="G$1" x="-22.86" y="58.42"/>
-<instance part="GND10" gate="1" x="-22.86" y="66.04"/>
 <instance part="GND11" gate="1" x="152.4" y="63.5"/>
 </instances>
@@
 </segment>
 <segment>
-<wire x1="-30.48" y1="68.58" x2="-22.86" y2="68.58" width="0.1524" layer="91"/>
-<pinref part="SV6" gate="A" pin="1"/>
-<pinref part="GND10" gate="1" pin="GND"/>
-</segment>
-<segment>
 <pinref part="SV5" gate="G$1" pin="39"/>
 <pinref part="GND11" gate="1" pin="GND"/>
@@
 </segment>
 <segment>
-<wire x1="-22.86" y1="76.2" x2="-22.86" y2="71.12" width="0.1524" layer="91"/>
-<wire x1="-22.86" y1="71.12" x2="-30.48" y2="71.12" width="0.1524" layer="91"/>
-<pinref part="+3V5" gate="G$1" pin="+3V3"/>
-<pinref part="SV6" gate="A" pin="2"/>
-</segment>
-<segment>
